File: PCB/V2.0/CacophonyV2/CacophonyV2.kicad_pcb (KiCad board)
At the start: 2 copper layers, 70.7 x 52.6 mm, 20 parts

Commit message: Added PCBv3
Parts:
- added D2: D, Diode_SMD:D_SMA, F.Cu at (172.8, 79.4)
- added D3: D, Diode_SMD:D_SMA, F.Cu at (187.9, 90.7)
- added D4: LED, LED_SMD:LED_0603_1608Metric, F.Cu at (195.8, 81.2)
- added D5: LED, LED_SMD:LED_0603_1608Metric, F.Cu at (195.8, 83.8)
- added R6: 150, Resistor_SMD:R_2512_6332Metric, F.Cu at (198.1, 72.6)
- added R7: 150, Resistor_SMD:R_2512_6332Metric, F.Cu at (183.1, 80.2)
- added REF**: MountingHole_3.2mm_M3, MountingHole:MountingHole_3.2mm_M3, F.Cu at (111.7, 98.3)
- added REF**: MountingHole_3.2mm_M3, MountingHole:MountingHole_3.2mm_M3, F.Cu at (170.0, 58.7)
- added REF**: MountingHole_3.2mm_M3, MountingHole:MountingHole_3.2mm_M3, F.Cu at (170.0, 101.1)
- added REF**: MountingHole_3.2mm_M3, MountingHole:MountingHole_3.2mm_M3, F.Cu at (111.7, 63.8)
Connections:
- B1 pad 3: +6V -> Net-(B1-Out+)
- B2 pad 3: +3.3V -> Net-(B2-Out+)
- C1 pad 1: +6V -> +5V
- C2 pad 1: +6V -> +5V
- C3 pad 1: +6V -> +5V
- C4 pad 1: +6V -> +5V
- S1 pad 2: +6V -> +5V
- S2 pad 2: +6V -> +5V
- U1 pad 1: +5V -> unconnected-(U1-5V-Pad1)
Routing:
- net +5V: track 30.0 -> 122.4 mm
- net +6V: track 35.8 -> 0.00 mm
- net Net-(B1-Out+): track 0.00 -> 5.88 mm
- net Net-(IC1-TX): track 48.2 -> 46.2 mm
- net Net-(IC1-RX): track 55.2 -> 54.4 mm
- net (no net): vias 2 -> 0
- added copper zone on F.Cu, net +5V
- removed copper zone on F.Cu, net +6V
